Commit message: add mycobot320gazebo-visual

File: mycobot_320m5_gazebo/arm_moveit/config/gazebo_firefighter.urdf (robot description, URDF)
Before this commit: robot firefighter, 16 links, 15 joints
Links:
- link base: geometry collision cylinder length=0.05 radius=0.053; visual mesh filename=package://mycobot_320_description/urdf/mycobot_320_m5_2022/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
- link gripper_base: geometry collision mesh filename=package://mycobot_320_description/urdf/mycobot_320_m5_2022/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; visual mesh filename=package://mycobot_320_description/urdf/mycobot_320_m5_2022/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
- link gripper_connection: geometry collision mesh filename=package://mycobot_320_description/urdf/mycobot_320_m5_2022/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; visual mesh filename=package://mycobot_320_description/urdf/mycobot_320_m5_2022/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
- link gripper_left1: geometry collision mesh filename=package://mycobot_320_description/urdf/mycobot_320_m5_2022/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; visual mesh filename=package://mycobot_320_description/urdf/mycobot_320_m5_2022/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
- link gripper_left2: geometry collision mesh filename=package://mycobot_320_description/urdf/mycobot_320_m5_2022/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; visual mesh filename=package://mycobot_320_description/urdf/mycobot_320_m5_2022/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
- link gripper_left3: geometry collision mesh filename=package://mycobot_320_description/urdf/mycobot_320_m5_2022/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; visual mesh filename=package://mycobot_320_description/urdf/mycobot_320_m5_2022/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
- link gripper_right1: geometry collision mesh filename=package://mycobot_320_description/urdf/mycobot_320_m5_2022/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; visual mesh filename=package://mycobot_320_description/urdf/mycobot_320_m5_2022/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
- link gripper_right2: geometry collision mesh filename=package://mycobot_320_description/urdf/mycobot_320_m5_2022/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; visual mesh filename=package://mycobot_320_description/urdf/mycobot_320_m5_2022/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
- link gripper_right3: geometry collision mesh filename=package://mycobot_320_description/urdf/mycobot_320_m5_2022/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; visual mesh filename=package://mycobot_320_description/urdf/mycobot_320_m5_2022/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
- link link1: geometry collision cylinder length=0.1 radius=0.033; visual mesh filename=package://mycobot_320_description/urdf/mycobot_320_m5_2022/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
- link link2: geometry collision cylinder length=0.15 radius=0.024; visual mesh filename=package://mycobot_320_description/urdf/mycobot_320_m5_2022/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
- link link3: geometry collision cylinder length=0.14 radius=0.0205; visual mesh filename=package://mycobot_320_description/urdf/mycobot_320_m5_2022/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
- link link4: geometry collision cylinder length=0.09 radius=0.024; visual mesh filename=package://mycobot_320_description/urdf/mycobot_320_m5_2022/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
- link link5: geometry collision cylinder length=0.1 radius=0.019; visual mesh filename=package://mycobot_320_description/urdf/mycobot_320_m5_2022/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
- link link6: geometry collision cylinder length=0.015 radius=0.026; visual mesh filename=package://mycobot_320_description/urdf/mycobot_320_m5_2022/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

File: mycobot_320m5_gazebo/demo_moveit/config/gazebo_ur5.urdf (robot description, URDF)
Before this commit: robot ur5, 21 links, 20 joints
Links:
- link base: geometry collision cylinder length=0.05 radius=0.053; visual mesh filename=package://mycobot_320_description/urdf/mycobot_320_m5_2022/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
- link camera_base_link: geometry collision mesh filename=package://mycobot_320_description/urdf/d435i.dae; visual mesh filename=package://mycobot_320_description/urdf/d435i.dae
- link gripper_base: geometry collision mesh filename=package://mycobot_320_description/urdf/mycobot_320_m5_2022/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; visual mesh filename=package://mycobot_320_description/urdf/mycobot_320_m5_2022/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
- link gripper_connection: geometry collision mesh filename=package://mycobot_320_description/urdf/mycobot_320_m5_2022/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; visual mesh filename=package://mycobot_320_description/urdf/mycobot_320_m5_2022/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
- link gripper_left1: geometry collision mesh filename=package://mycobot_320_description/urdf/mycobot_320_m5_2022/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; visual mesh filename=package://mycobot_320_description/urdf/mycobot_320_m5_2022/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
- link gripper_left2: geometry collision mesh filename=package://mycobot_320_description/urdf/mycobot_320_m5_2022/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; visual mesh filename=package://mycobot_320_description/urdf/mycobot_320_m5_2022/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
- link gripper_left3: geometry collision mesh filename=package://mycobot_320_description/urdf/mycobot_320_m5_2022/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; visual mesh filename=package://mycobot_320_description/urdf/mycobot_320_m5_2022/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
- link gripper_right1: geometry collision mesh filename=package://mycobot_320_description/urdf/mycobot_320_m5_2022/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; visual mesh filename=package://mycobot_320_description/urdf/mycobot_320_m5_2022/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
- link gripper_right2: geometry collision mesh filename=package://mycobot_320_description/urdf/mycobot_320_m5_2022/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; visual mesh filename=package://mycobot_320_description/urdf/mycobot_320_m5_2022/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
- link gripper_right3: geometry collision mesh filename=package://mycobot_320_description/urdf/mycobot_320_m5_2022/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; visual mesh filename=package://mycobot_320_description/urdf/mycobot_320_m5_2022/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
- link link1: geometry collision cylinder length=0.1 radius=0.033; visual mesh filename=package://mycobot_320_description/urdf/mycobot_320_m5_2022/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
- link link2: geometry collision cylinder length=0.15 radius=0.024; visual mesh filename=package://mycobot_320_description/urdf/mycobot_320_m5_2022/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
- link link3: geometry collision cylinder length=0.14 radius=0.0205; visual mesh filename=package://mycobot_320_description/urdf/mycobot_320_m5_2022/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
- link link4: geometry collision cylinder length=0.09 radius=0.024; visual mesh filename=package://mycobot_320_description/urdf/mycobot_320_m5_2022/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
- link link5: geometry collision cylinder length=0.1 radius=0.019; visual mesh filename=package://mycobot_320_description/urdf/mycobot_320_m5_2022/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
- link link6: geometry collision cylinder length=0.015 radius=0.026; visual mesh filename=package://mycobot_320_description/urdf/mycobot_320_m5_2022/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
